Commit message: modified robot_bullet+custom environment begin
auto set number of actuated joints (all prismatic and revolute) and number of observed links(all)
copied gym env pendolum v0 as template
fixed path pendulum urdf

File: urdf/single_pendulum.urdf (robot description, URDF)
Before this commit: robot 1dof_planar, 3 links, 2 joints
Links:
- link base_link: geometry collision mesh filename=/home/pasquale/Desktop/thesis/stl/base_link.stl; visual mesh filename=/home/pasquale/Desktop/thesis/stl/base_link.stl
- link link1: geometry collision mesh filename=/home/pasquale/Desktop/thesis/stl/link1.stl; visual mesh filename=/home/pasquale/Desktop/thesis/stl/link1.stl

Commit message: added custom policy file

File: urdf/single_pendulum.urdf (robot description, URDF)
Before this commit: robot 1dof_planar, 3 links, 2 joints
Joints:
- joint joint1: limit effort=10 velocity=50 -> effort=1000 velocity=1000
