Commit message: fixed step issue during evaluation

File: urdf/double_pendulum.urdf (robot description, URDF)
Before this commit: robot 2dof_planar, 4 links, 3 joints
Joints:
- joint joint1: origin xyz=0.0060872 0 0.035 rpy=3.1416 0 0 -> xyz=0.0060872 0 0.035 rpy=3.141592 0 0

File: urdf/single_pendulum.urdf (robot description, URDF)
Before this commit: robot 1dof_planar, 3 links, 2 joints
Joints:
- joint joint1: origin xyz=0.0060872 0 0.035 rpy=3.1416 0 0 -> xyz=0.0060872 0 0.035 rpy=3.14192 0 0
